File: KiCad/UA-1_v1/UA-1_v1.kicad_pcb (KiCad board)
At the start: 2 copper layers, 207 x 107.2 mm, 44 parts, among them IC1 74LVC4245APW,112, J1 RF_base, J2 RF_base_gnd, J3 12V, J4 UART_FW, J5 RF_mine, J6 RF_mine_gnd, U1 MP-N, U2 AMS1117-3.3, U3 ESP32-WROOM-32E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

Commit message: add pls1-3
Parts:
- JP1: value FW -> PLS-3
Changed lines of the file:
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@@
 			)
 		)
-		(property "Value" "FW"
+		(property "Value" "PLS-3"
 			(at 0 7.41 0)
 			(layer "F.Fab")
@@
 		(property ki_fp_filters "Jumper* TestPoint*3Pads* TestPoint*Bridge*")
 		(sheetname "Корневой лист")
-		(sheetfile "SmartAtt.kicad_sch")
-		(attr through_hole exclude_from_bom)
+		(sheetfile "UA-1_v1.kicad_sch")
+		(attr through_hole)
 		(fp_line
 			(start -1.33 -1.33)
@@
 		)
 		(sheetname "Корневой лист")
-		(sheetfile "SmartAtt.kicad_sch")
+		(sheetfile "UA-1_v1.kicad_sch")
 		(attr through_hole)
 		(fp_rect
@@
 			(net 5 "+5V")
 			(pinfunction "Vout")
-			(pintype "passive")
+			(pintype "power_out")
 		)
 		(pad "4" thru_hole circle
@@
 		)
 		(sheetname "Корневой лист")
-		(sheetfile "SmartAtt.kicad_sch")
+		(sheetfile "UA-1_v1.kicad_sch")
 		(attr through_hole)
 		(fp_rect
@@
 		(property ki_fp_filters "Connector*:*_1x??_*")
 		(sheetname "Корневой лист")
-		(sheetfile "SmartAtt.kicad_sch")
+		(sheetfile "UA-1_v1.kicad_sch")
 		(attr exclude_from_pos_files)
 		(fp_line
@@
 		(property ki_fp_filters "*Buzzer*")
 		(sheetname "Корневой лист")
-		(sheetfile "SmartAtt.kicad_sch")
+		(sheetfile "UA-1_v1.kicad_sch")
 		(attr through_hole)
 		(fp_rect
@@
 		(property ki_fp_filters "Connector*:*_1x??_*")
 		(sheetname "Корневой лист")
-		(sheetfile "SmartAtt.kicad_sch")
+		(sheetfile "UA-1_v1.kicad_sch")
 		(attr exclude_from_pos_files)
 		(fp_line
@@
 		(property ki_fp_filters "Connector*:*_1x??_*")
 		(sheetname "Корневой лист")
-		(sheetfile "SmartAtt.kicad_sch")
+		(sheetfile "UA-1_v1.kicad_sch")
 		(attr exclude_from_pos_files)
 		(fp_line
@@
 		(property ki_fp_filters "LED* LED_SMD:* LED_THT:*")
 		(sheetname "Корневой лист")
-		(sheetfile "SmartAtt.kicad_sch")
+		(sheetfile "UA-1_v1.kicad_sch")
 		(attr smd)
 		(fp_line
@@
 		)
 		(sheetname "Корневой лист")
-		(sheetfile "SmartAtt.kicad_sch")
+		(sheetfile "UA-1_v1.kicad_sch")
 		(attr smd)
 		(fp_rect
@@
 		(property ki_fp_filters "Connector*:*_1x??_*")
 		(sheetname "Корневой лист")
-		(sheetfile "SmartAtt.kicad_sch")
+		(sheetfile "UA-1_v1.kicad_sch")
 		(attr exclude_from_pos_files)
 		(fp_line
@@
 		(property ki_fp_filters "Connector*:*_1x??_*")
 		(sheetname "Корневой лист")
-		(sheetfile "SmartAtt.kicad_sch")
+		(sheetfile "UA-1_v1.kicad_sch")
 		(attr through_hole)
 		(fp_line
@@
 		(property ki_fp_filters "Connector*:*_1x??_*")
 		(sheetname "Корневой лист")
-		(sheetfile "SmartAtt.kicad_sch")
+		(sheetfile "UA-1_v1.kicad_sch")
 		(attr through_hole)
 		(fp_line
@@
 		(property ki_fp_filters "R_*")
 		(sheetname "Корневой лист")
-		(sheetfile "SmartAtt.kicad_sch")
+		(sheetfile "UA-1_v1.kicad_sch")
 		(attr smd)
 		(fp_line
@@
 		(property ki_fp_filters "TO-???* *_Diode_* *SingleDiode* D_*")
 		(sheetname "Корневой лист")
-		(sheetfile "SmartAtt.kicad_sch")
+		(sheetfile "UA-1_v1.kicad_sch")
 		(attr smd)
 		(fp_line
@@
 		(property ki_fp_filters "C_*")
 		(sheetname "Корневой лист")
-		(sheetfile "SmartAtt.kicad_sch")
+		(sheetfile "UA-1_v1.kicad_sch")
 		(attr smd)
 		(fp_line
@@
 		(property ki_fp_filters "C_*")
 		(sheetname "Корневой лист")
-		(sheetfile "SmartAtt.kicad_sch")
+		(sheetfile "UA-1_v1.kicad_sch")
 		(attr through_hole)
 		(fp_line
@@
 		(property ki_fp_filters "CP_*")
 		(sheetname "Корневой лист")
-		(sheetfile "SmartAtt.kicad_sch")
+		(sheetfile "UA-1_v1.kicad_sch")
 		(attr smd)
 		(fp_line
@@
 		(property ki_fp_filters "R_*")
 		(sheetname "Корневой лист")
-		(sheetfile "SmartAtt.kicad_sch")
+		(sheetfile "UA-1_v1.kicad_sch")
 		(attr smd)
 		(fp_line
@@
 		(property ki_fp_filters "C_*")
 		(sheetname "Корневой лист")
-		(sheetfile "SmartAtt.kicad_sch")
+		(sheetfile "UA-1_v1.kicad_sch")
 		(attr smd)
 		(fp_line
@@
 		(property ki_fp_filters "CP_*")
 		(sheetname "Корневой лист")
-		(sheetfile "SmartAtt.kicad_sch")
+		(sheetfile "UA-1_v1.kicad_sch")
 		(attr smd)
 		(fp_line
@@
 		(property ki_fp_filters "R_*")
 		(sheetname "Корневой лист")
-		(sheetfile "SmartAtt.kicad_sch")
+		(sheetfile "UA-1_v1.kicad_sch")
 		(attr smd)
 		(fp_line
@@
 		(property ki_fp_filters "C_*")
 		(sheetname "Корневой лист")
-		(sheetfile "SmartAtt.kicad_sch")
+		(sheetfile "UA-1_v1.kicad_sch")
 		(attr smd)
 		(fp_line
@@
 		(property ki_fp_filters "TO-???* *_Diode_* *SingleDiode* D_*")
 		(sheetname "Корневой лист")
-		(sheetfile "SmartAtt.kicad_sch")
+		(sheetfile "UA-1_v1.kicad_sch")
 		(attr smd)
 		(fp_line
@@
 		(property ki_fp_filters "CP_*")
 		(sheetname "Корневой лист")
-		(sheetfile "SmartAtt.kicad_sch")
+		(sheetfile "UA-1_v1.kicad_sch")
 		(attr smd)
 		(fp_line
@@
 		(property ki_fp_filters "ESP32?WROOM?32D*")
 		(sheetname "Корневой лист")
-		(sheetfile "SmartAtt.kicad_sch")
+		(sheetfile "UA-1_v1.kicad_sch")
 		(attr smd)
 		(fp_line
@@
 		(property ki_fp_filters "TO-???* *_Diode_* *SingleDiode* D_*")
 		(sheetname "Корневой лист")
-		(sheetfile "SmartAtt.kicad_sch")
+		(sheetfile "UA-1_v1.kicad_sch")
 		(attr smd)
 		(fp_line
@@
 		(property ki_fp_filters "SOT?223*TabPin2*")
 		(sheetname "Корневой лист")
-		(sheetfile "SmartAtt.kicad_sch")
+		(sheetfile "UA-1_v1.kicad_sch")
 		(attr smd)
 		(fp_line
@@
 		)
 		(sheetname "Корневой лист")
-		(sheetfile "SmartAtt.kicad_sch")
+		(sheetfile "UA-1_v1.kicad_sch")
 		(attr smd)
 		(fp_line
@@
 		(property ki_fp_filters "R_*")
 		(sheetname "Корневой лист")
-		(sheetfile "SmartAtt.kicad_sch")
+		(sheetfile "UA-1_v1.kicad_sch")
 		(attr smd)
 		(fp_line
@@
 		(property ki_fp_filters "Choke_* *Coil* Inductor_* L_*")
 		(sheetname "Корневой лист")
-		(sheetfile "SmartAtt.kicad_sch")
+		(sheetfile "UA-1_v1.kicad_sch")
 		(attr through_hole)
 		(fp_line
@@
 		(property ki_fp_filters "CP_*")
 		(sheetname "Корневой лист")
-		(sheetfile "SmartAtt.kicad_sch")
+		(sheetfile "UA-1_v1.kicad_sch")
 		(attr smd)
 		(fp_line
@@
 		(property ki_fp_filters "R_*")
 		(sheetname "Корневой лист")
-		(sheetfile "SmartAtt.kicad_sch")
+		(sheetfile "UA-1_v1.kicad_sch")
 		(attr smd)
 		(fp_line
@@
 		(property ki_fp_filters "C_*")
 		(sheetname "Корневой лист")
-		(sheetfile "SmartAtt.kicad_sch")
+		(sheetfile "UA-1_v1.kicad_sch")
 		(attr smd)
 		(fp_line
@@
 		(property ki_fp_filters "CP_*")
 		(sheetname "Корневой лист")
-		(sheetfile "SmartAtt.kicad_sch")
+		(sheetfile "UA-1_v1.kicad_sch")
 		(attr smd)
 		(fp_line
@@
 		(property ki_fp_filters "Choke_* *Coil* Inductor_* L_*")
 		(sheetname "Корневой лист")
-		(sheetfile "SmartAtt.kicad_sch")
+		(sheetfile "UA-1_v1.kicad_sch")
 		(attr through_hole)
 		(fp_line
@@
 		(property ki_fp_filters "CP_*")
 		(sheetname "Корневой лист")
-		(sheetfile "SmartAtt.kicad_sch")
+		(sheetfile "UA-1_v1.kicad_sch")
 		(attr smd)
 		(fp_line
@@
 		(property ki_fp_filters "C_*")
 		(sheetname "Корневой лист")
-		(sheetfile "SmartAtt.kicad_sch")
+		(sheetfile "UA-1_v1.kicad_sch")
 		(attr smd)
 		(fp_line
@@
 		(property ki_fp_filters "R_*")
 		(sheetname "Корневой лист")
-		(sheetfile "SmartAtt.kicad_sch")
+		(sheetfile "UA-1_v1.kicad_sch")
 		(attr smd)
 		(fp_line
@@
 		)
 		(sheetname "Корневой лист")
-		(sheetfile "SmartAtt.kicad_sch")
+		(sheetfile "UA-1_v1.kicad_sch")
 		(attr smd)
 		(fp_line
@@
 		(property ki_fp_filters "C_*")
 		(sheetname "Корневой лист")
-		(sheetfile "SmartAtt.kicad_sch")
+		(sheetfile "UA-1_v1.kicad_sch")
 		(attr smd)
 		(fp_line
@@
 		(property ki_fp_filters "C_*")
 		(sheetname "Корневой лист")
-		(sheetfile "SmartAtt.kicad_sch")
+		(sheetfile "UA-1_v1.kicad_sch")
 		(attr smd)
 		(fp_line
@@
 		(property ki_fp_filters "C_*")
 		(sheetname "Корневой лист")
-		(sheetfile "SmartAtt.kicad_sch")
+		(sheetfile "UA-1_v1.kicad_sch")
 		(attr through_hole)
 		(fp_line
@@
 		(property ki_fp_filters "R_*")
 		(sheetname "Корневой лист")
-		(sheetfile "SmartAtt.kicad_sch")
+		(sheetfile "UA-1_v1.kicad_sch")
 		(attr smd dnp)
 		(fp_line
@@
 		(property ki_fp_filters "CP_*")
 		(sheetname "Корневой лист")
-		(sheetfile "SmartAtt.kicad_sch")
+		(sheetfile "UA-1_v1.kicad_sch")
 		(attr smd)
 		(fp_line
