File: KiCad/UA-1_v2/UA-1_v2.kicad_pcb (KiCad board)
At the start: 2 copper layers, 207 x 107.2 mm, 44 parts, among them IC1 74LVC4245APW,112, J1 RF_base, J2 RF_base_gnd, J3 12V, J4 UART_FW, J5 RF_mine, J6 RF_mine_gnd, U1 MP-N, U2 AMS1117-3.3, U3 ESP32-WROOM-32E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

Commit message: v2 prod
Parts:
- moved C1 48.1 mm to (101.3, 90.8)
- moved C16 41.7 mm to (212.8, 90.7)
- moved R7 4.43 mm to (121.8, 54.1)
Connections:
- BZ1 pad 1: Net-(BZ1-+) -> GND
- BZ1 pad 2: GND -> Net-(BZ1--)
- R7 pad 2: Net-(BZ1-+) -> Net-(BZ1--)
Routing:
- net Net-(J1-Pin_1): track 75.4 -> 27.3 mm
- net Net-(U4-RF1): track 4.16 -> 52.3 mm
- net Net-(U4-RF2): track 3.76 -> 45.4 mm
- net Net-(J5-Pin_1): track 61.2 -> 19.6 mm
- net Net-(BZ1--): track 0.00 -> 6.25 mm
- net /BUZ: track 118.0 -> 112.8 mm
- net Net-(BZ1-+): track 4.30 -> 0.00 mm
- net +3.3V: track 218.4 -> 218.5 mm, vias 5 -> 7
- net +5V: vias 5 -> 7
Other:
- board text added: "+3"
- board text added: "FW"
- board text added: "GND"
- board text added: "RX"
- board text added: "TX"
- board text added: "УА-1 v2"
- board text removed: "УА-1 v1"
