File: KiCad/UA-1_v2/UA-1_v2.kicad_sch (KiCad schematic)
At the start: 44 parts, among them IC1 74LVC4245APW,112, J1 RF_base, J2 RF_base_gnd, J3 12V, J4 UART_FW, J5 RF_mine, J6 RF_mine_gnd, U1 MP-N, U2 AMS1117-3.3, U3 ESP32-WROOM-32E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

Commit message: v2 prod
Connections:
- net GND: now also BZ1.1 (+); no longer BZ1.2 (-)
- net at R7.2: now also BZ1.2 (-); no longer BZ1.1 (+)
Changed lines of the file:
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@@
 		(lib_id "Device:Buzzer")
 		(at 255.27 39.37 0)
+		(mirror x)
 		(unit 1)
 		(exclude_from_sim no)
@@
 		(fields_autoplaced yes)
 		(property "Reference" "BZ1"
-			(at 259.08 38.0999 0)
+			(at 259.08 40.6401 0)
 			(effects
 				(font
@@
 		)
 		(property "Value" "Buzzer"
-			(at 259.08 40.6399 0)
+			(at 259.08 38.1001 0)
 			(effects
 				(font
@@
 		)
 		(property "Footprint" "Alexeyj4:HC0903A"
-			(at 254.635 36.83 90)
+			(at 254.635 41.91 90)
 			(effects
 				(font
@@
 		)
 		(property "Datasheet" "~"
-			(at 254.635 36.83 90)
+			(at 254.635 41.91 90)
 			(effects
 				(font
